Commit message: map generated

File: src/mobile_robot/model/flap_bot.xacro (robot description, xacro)
@@ -1,27 +1,28 @@
 <?xml version="1.0"?>
-<robot name="flap_bot" xmlns:xacro="http://www.ros.org/wiki/xacro">
-  <!-- ========================== -->
-  <!-- PROPERTIES -->
-  <!-- ========================== -->
-  <xacro:property name="base_length" value="0.6"/>
-  <xacro:property name="base_width" value="0.4"/>
-  <xacro:property name="base_height" value="0.2"/>
-  <xacro:property name="wheel_radius" value="0.1"/>
-  <xacro:property name="wheel_length" value="0.05"/>
-  <xacro:property name="caster_radius" value="0.05"/>
+<robot name="flap_tb3_bot" xmlns:xacro="http://www.ros.org/wiki/xacro">
+  <!-- ========================== -->
+  <!-- PROPERTIES (SCALED UP)    -->
+  <!-- ========================== -->
+  <!-- Robot size increased ~30% -->
+  <xacro:property name="base_length" value="0.75"/>
+  <xacro:property name="base_width"  value="0.55"/>
+  <xacro:property name="base_height" value="0.25"/>
+  <xacro:property name="wheel_radius"  value="0.12"/>
+  <xacro:property name="wheel_length"  value="0.06"/>
+  <xacro:property name="caster_radius" value="0.06"/>
   <xacro:property name="pi" value="3.14159265359"/>
-  <!-- Flap (finger) dimensions -->
-  <xacro:property name="finger_length" value="0.2"/>
-  <xacro:property name="finger_width" value="0.03"/>
-  <xacro:property name="finger_height" value="0.08"/>
-  <!-- LIDAR dimensions -->
-  <xacro:property name="lidar_radius" value="0.07"/>
-  <xacro:property name="lidar_length" value="0.04"/>
-  <xacro:property name="lidar_height_offset" value="${base_height/2.0 + 0.15}"/>
+  <!-- Flap (finger) dimensions - LONGER + WIDER -->
+  <xacro:property name="finger_length" value="0.40"/>  <!-- was 0.2 -->
+  <xacro:property name="finger_width"  value="0.06"/>  <!-- was 0.03 -->
+  <xacro:property name="finger_height" value="0.10"/>  <!-- slightly taller -->
+  <!-- LIDAR dimensions (slightly larger) -->
+  <xacro:property name="lidar_radius"        value="0.08"/>
+  <xacro:property name="lidar_length"        value="0.05"/>
+  <xacro:property name="lidar_height_offset" value="${base_height/2.0 + 0.18}"/>
   <!-- Control -->
   <xacro:property name="max_linear_acceleration" value="10"/>
   <xacro:property name="wheel_separation" value="${base_width + wheel_length}"/>
   <!-- ========================== -->
-  <!-- MATERIALS -->
+  <!-- MATERIALS                  -->
   <!-- ========================== -->
   <material name="blue">
@@ -35,8 +36,8 @@
   </material>
   <!-- ========================== -->
-  <!-- BASE & FOOTPRINT -->
-  <!-- ========================== -->
-  <link name="base_footprint"/>
-  <link name="base_link">
+  <!-- BASE & FOOTPRINT           -->
+  <!-- ========================== -->
+  <link name="base_link"/>
+  <link name="chassis">
     <visual>
       <origin xyz="0 0 ${base_height/2.0}" rpy="0 0 0"/>
@@ -54,16 +55,16 @@
     <inertial>
       <origin xyz="0 0 ${base_height/2.0}" rpy="0 0 0"/>
-      <mass value="5.0"/>
-      <inertia ixx="0.1" iyy="0.1" izz="0.1" ixy="0" ixz="0" iyz="0"/>
-    </inertial>
-  </link>
-  <!-- Raise base so wheels touch ground -->
-  <joint name="robot_base_joint" type="fixed">
-    <parent link="base_footprint"/>
-    <child link="base_link"/>
+      <mass value="7.0"/>
+      <inertia ixx="0.2" iyy="0.2" izz="0.2" ixy="0" ixz="0" iyz="0"/>
+    </inertial>
+  </link>
+<!-- Raise base so wheels touch ground -->
+  <joint name="chassis_joint" type="fixed">
+    <parent link="base_link"/>  <!-- This was changed from world to base_link -->
+    <child link="chassis"/>
     <origin xyz="0 0 ${wheel_radius}"/>
   </joint>
   <!-- ========================== -->
-  <!-- WHEEL MACRO -->
+  <!-- WHEEL MACRO                -->
   <!-- ========================== -->
   <xacro:macro name="wheel_link" params="prefix">
@@ -84,6 +85,6 @@
       <inertial>
         <origin xyz="0 0 0"/>
-        <mass value="0.2"/>
-        <inertia ixx="0.001" iyy="0.001" izz="0.001" ixy="0" ixz="0" iyz="0"/>
+        <mass value="0.3"/>
+        <inertia ixx="0.002" iyy="0.002" izz="0.002" ixy="0" ixz="0" iyz="0"/>
       </inertial>
     </link>
@@ -96,5 +97,5 @@
   <xacro:wheel_link prefix="left"/>
   <!-- ========================== -->
-  <!-- CASTER WHEEL -->
+  <!-- CASTER WHEEL               -->
   <!-- ========================== -->
   <link name="caster_wheel_link">
@@ -112,6 +113,6 @@
     <inertial>
       <origin xyz="0 0 0"/>
-      <mass value="0.05"/>
-      <inertia ixx="0.0005" iyy="0.0005" izz="0.0005" ixy="0" ixz="0" iyz="0"/>
+      <mass value="0.07"/>
+      <inertia ixx="0.0007" iyy="0.0007" izz="0.0007" ixy="0" ixz="0" iyz="0"/>
     </inertial>
   </link>
@@ -121,9 +122,10 @@
   </gazebo>
   <!-- ========================== -->
-  <!-- FLAPS / FINGERS -->
+  <!-- FLAPS / FINGERS (WIDER)    -->
   <!-- ========================== -->
   <link name="left_flap_link">
     <visual>
-      <origin xyz="0 0 0" rpy="0 0 0.2"/>
+      <!-- rotated slightly outward (counter-clockwise) -->
+      <origin xyz="0 0 0" rpy="0 0 0.25"/>
       <geometry>
         <box size="${finger_length} ${finger_width} ${finger_height}"/>
@@ -132,5 +134,5 @@
     </visual>
     <collision>
-      <origin xyz="0 0 0" rpy="0 0 0.2"/>
+      <origin xyz="0 0 0" rpy="0 0 0.25"/>
       <geometry>
         <box size="${finger_length} ${finger_width} ${finger_height}"/>
@@ -138,12 +140,13 @@
     </collision>
     <inertial>
-      <origin xyz="${finger_length/2} ${finger_width/2} ${finger_height/2}"/>
-      <mass value="0.07"/>
-      <inertia ixx="0.00005" iyy="0.00005" izz="0.00006" ixy="0" ixz="0" iyz="0"/>
+      <origin xyz="${finger_length/2} 0 ${finger_height/2}"/>
+      <mass value="0.10"/>
+      <inertia ixx="0.00008" iyy="0.00008" izz="0.00009" ixy="0" ixz="0" iyz="0"/>
     </inertial>
   </link>
   <link name="right_flap_link">
     <visual>
-      <origin xyz="0 0 0" rpy="0 0 -0.2"/>
+      <!-- rotated slightly outward (clockwise) -->
+      <origin xyz="0 0 0" rpy="0 0 -0.25"/>
       <geometry>
         <box size="${finger_length} ${finger_width} ${finger_height}"/>
@@ -152,5 +155,5 @@
     </visual>
     <collision>
-      <origin xyz="0 0 0" rpy="0 0 -0.2"/>
+      <origin xyz="0 0 0" rpy="0 0 -0.25"/>
       <geometry>
         <box size="${finger_length} ${finger_width} ${finger_height}"/>
@@ -158,11 +161,11 @@
     </collision>
     <inertial>
-      <origin xyz="${finger_length/2} ${finger_width/2} ${finger_height/2}"/>
-      <mass value="0.07"/>
-      <inertia ixx="0.00005" iyy="0.00005" izz="0.00006" ixy="0" ixz="0" iyz="0"/>
-    </inertial>
-  </link>
-  <!-- ========================== -->
-  <!-- LIDAR -->
+      <origin xyz="${finger_length/2} 0 ${finger_height/2}"/>
+      <mass value="0.10"/>
+      <inertia ixx="0.00008" iyy="0.00008" izz="0.00009" ixy="0" ixz="0" iyz="0"/>
+    </inertial>
+  </link>
+  <!-- ========================== -->
+  <!-- LIDAR                      -->
   <!-- ========================== -->
   <link name="lidar_link">
@@ -181,28 +184,38 @@
     <inertial>
       <origin xyz="0 0 0"/>
-      <mass value="0.1"/>
-      <inertia ixx="0.0005" iyy="0.0005" izz="0.0005" ixy="0" ixz="0" iyz="0"/>
-    </inertial>
-  </link>
+      <mass value="0.15"/>
+      <inertia ixx="0.0007" iyy="0.0007" izz="0.0007" ixy="0" ixz="0" iyz="0"/>
+    </inertial>
+  </link>
+  <!-- LIDAR sensor: Laser system, frame_id = lidar_link -->
   <gazebo reference="lidar_link">
-    <sensor name="laser_sensor" type="gpu_lidar">
-      <topic>lidar</topic>
+    <sensor name='gpu_lidar' type='gpu_lidar'>
+      <always_on>true</always_on>
+      <visualize>true</visualize>
       <pose>0 0 0 0 0 0</pose>
-      <update_rate>10</update_rate>
-      <ray>
+      <update_rate>5</update_rate>
+      <topic>scan</topic>
+      <gz_frame_id>lidar_link</gz_frame_id>
+      <lidar>
         <scan>
           <horizontal>
             <samples>640</samples>
             <resolution>1</resolution>
-            <min_angle>-2.2689</min_angle>
-            <max_angle> 2.2689</max_angle>
+            <min_angle>-3.1416</min_angle>
+            <max_angle>3.1416</max_angle>
           </horizontal>
         </scan>
         <range>
-          <min>0.1</min>
-          <max>10.0</max>
+          <min>0.5</min>
+          <max>8.0</max>
           <resolution>0.01</resolution>
         </range>
-      </ray>
+        <noise>
+          <type>gaussian</type>
+          <mean>0.0</mean>
+          <stddev>0.01</stddev>
+        </noise>
+        <frame_id>laser_link</frame_id>
+      </lidar>
       <always_on>1</always_on>
       <visualize>true</visualize>
@@ -210,5 +223,5 @@
   </gazebo>
   <!-- ========================== -->
-  <!-- JOINTS -->
+  <!-- JOINTS                     -->
   <!-- ========================== -->
   <!-- Wheels -->
@@ -227,20 +240,28 @@
   <!-- Caster -->
   <joint name="base_caster_wheel_joint" type="fixed">
-    <parent link="base_link"/>
+    <parent link="chassis"/>
     <child link="caster_wheel_link"/>
     <origin xyz="${base_length/3} 0 ${-(wheel_radius - caster_radius)}"/>
   </joint>
-  <!-- Flaps -->
+  <!-- Flaps
+       NOTE: y = +/- (base_width/2 - finger_width/2)
+       so the flaps sit almost at the outer edges, giving more useful width.
+       Limits remain 0..1.2 rad so teleop code does NOT need changes.
+  -->
   <joint name="left_flap_joint" type="revolute">
-    <parent link="base_link"/>
+    <parent link="chassis"/>
     <child link="left_flap_link"/>
-    <origin xyz="${base_length/2 + finger_length/2} ${base_width/4} ${finger_height/2}" rpy="0 0 0"/>
+    <origin
+      xyz="${base_length/2 + finger_length/2} ${base_width/2 - finger_width/2} ${finger_height/2}"
+      rpy="0 0 0"/>
     <axis xyz="0 0 -1"/>
     <limit lower="0" upper="1.2" effort="10" velocity="1.5"/>
   </joint>
   <joint name="right_flap_joint" type="revolute">
-    <parent link="base_link"/>
+    <parent link="chassis"/>
     <child link="right_flap_link"/>
-    <origin xyz="${base_length/2 + finger_length/2} ${-base_width/4} ${finger_height/2}" rpy="0 0 0"/>
+    <origin
+      xyz="${base_length/2 + finger_length/2} ${-(base_width/2 - finger_width/2)} ${finger_height/2}"
+      rpy="0 0 0"/>
     <axis xyz="0 0 1"/>
     <limit lower="0" upper="1.2" effort="10" velocity="1.5"/>
@@ -248,10 +269,27 @@
   <!-- LIDAR joint -->
   <joint name="lidar_joint" type="fixed">
-    <parent link="base_link"/>
+    <parent link="chassis"/>
     <child link="lidar_link"/>
     <origin xyz="0 0 ${lidar_height_offset}"/>
   </joint>
-  <!-- ========================== -->
-  <!-- GAZEBO PLUGINS -->
+<!-- IMU Sensor -->
+  <joint name="imu_joint" type="fixed">
+    <origin xyz="0 0 0" rpy="0 0 0" />
+    <parent link="base_link"/>
+    <child link="imu_link" />
+  </joint>
+  <gazebo reference="imu_link">
+    <sensor name="imu" type="imu">
+      <always_on>true</always_on>
+      <update_rate>200</update_rate>
+      <visualize>true</visualize>
+      <topic>imu</topic>
+      <enable_metrics>true</enable_metrics>
+      <gz_frame_id>imu_link</gz_frame_id>
+    </sensor>
+  </gazebo>
+  <link name="imu_link" />
+  <!-- ========================== -->
+  <!-- GAZEBO PLUGINS             -->
   <!-- ========================== -->
   <gazebo>
@@ -263,7 +301,5 @@
       <wheel_radius>${wheel_radius}</wheel_radius>
       <max_linear_acceleration>${max_linear_acceleration}</max_linear_acceleration>
-      <odom_publish_frequency>100</odom_publish_frequency>
       <topic>cmd_vel</topic>
-      <odom_topic>odom</odom_topic>
     </plugin>
     <!-- Joint state publisher -->
@@ -275,5 +311,5 @@
       <joint_name>right_flap_joint</joint_name>
     </plugin>
-    <!-- Flap position controllers (THIS is the important fix) -->
+    <!-- Flap position controllers (topics unchanged) -->
     <plugin
       filename="gz-sim-joint-position-controller-system"
@@ -290,4 +326,14 @@
       <p_gain>50.0</p_gain>
     </plugin>
+    <plugin
+      filename="gz-sim-odometry-publisher-system"
+      name="gz::sim::systems::OdometryPublisher">
+      <odom_frame>odom</odom_frame>
+      <robot_base_frame>base_link</robot_base_frame>
+      <odom_publish_frequency>50</odom_publish_frequency>
+      <odom_topic>/odom</odom_topic>
+      <tf_topic>/tf</tf_topic>
+      <dimensions>2</dimensions>
+    </plugin>
   </gazebo>
 </robot>

File: src/mobile_robot/model/flap_tb3_bot.xacro (robot description, xacro)
@@ -61,5 +61,5 @@
 <!-- Raise base so wheels touch ground -->
   <joint name="robot_base_joint" type="fixed">
-    <parent link="base_footprint"/>  <!-- This was changed from world to base_link -->
+    <parent link="base_footprint"/>
     <child link="base_link"/>
     <origin xyz="0 0 ${wheel_radius}"/>
@@ -205,10 +205,4 @@
             <max_angle>3.1416</max_angle>
           </horizontal>
-          <vertical>
-            <samples>1</samples>
-            <resolution>0.01</resolution>
-            <min_angle>0</min_angle>
-            <max_angle>0</max_angle>
-          </vertical>
         </scan>
         <range>
@@ -217,5 +211,13 @@
           <resolution>0.01</resolution>
         </range>
+        <noise>
+          <type>gaussian</type>
+          <mean>0.0</mean>
+          <stddev>0.01</stddev>
+        </noise>
+        <frame_id>lidar_link</frame_id>
       </lidar>
+      <always_on>1</always_on>
+      <visualize>true</visualize>
     </sensor>
   </gazebo>
@@ -271,4 +273,21 @@
     <origin xyz="0 0 ${lidar_height_offset}"/>
   </joint>
+<!-- IMU Sensor -->
+  <joint name="imu_joint" type="fixed">
+    <origin xyz="0 0 0" rpy="0 0 0" />
+    <parent link="base_link"/>
+    <child link="imu_link" />
+  </joint>
+  <gazebo reference="imu_link">
+    <sensor name="imu" type="imu">
+      <always_on>true</always_on>
+      <update_rate>200</update_rate>
+      <visualize>true</visualize>
+      <topic>imu</topic>
+      <enable_metrics>true</enable_metrics>
+      <gz_frame_id>imu_link</gz_frame_id>
+    </sensor>
+  </gazebo>
+  <link name="imu_link" />
   <!-- ========================== -->
   <!-- GAZEBO PLUGINS             -->
@@ -282,12 +301,5 @@
       <wheel_radius>${wheel_radius}</wheel_radius>
       <max_linear_acceleration>${max_linear_acceleration}</max_linear_acceleration>
-      <odom_publish_frequency>100</odom_publish_frequency>
       <topic>cmd_vel</topic>
-      <publish_odom>true</publish_odom>
-      <publish_wheel_tf>true</publish_wheel_tf>
-      <publish_odom_tf>true</publish_odom_tf>
-      <odom_topic>odom</odom_topic>
-      <frame_id>odom</frame_id>
-      <child_frame_id>base_footprint</child_frame_id>
     </plugin>
     <!-- Joint state publisher -->
@@ -314,4 +326,14 @@
       <p_gain>50.0</p_gain>
     </plugin>
+    <plugin
+      filename="gz-sim-odometry-publisher-system"
+      name="gz::sim::systems::OdometryPublisher">
+      <odom_frame>odom</odom_frame>
+      <robot_base_frame>base_footprint</robot_base_frame>
+      <odom_publish_frequency>50</odom_publish_frequency>
+      <odom_topic>/odom</odom_topic>
+      <tf_topic>/tf</tf_topic>
+      <dimensions>2</dimensions>
+    </plugin>
   </gazebo>
 </robot>
