Commit message: SLAM in progress

File: src/mobile_robot/model/flap_tb3_bot.xacro (robot description, xacro)
@@ -59,7 +59,7 @@
     </inertial>
   </link>
-  <!-- Raise base so wheels touch ground -->
+<!-- Raise base so wheels touch ground -->
   <joint name="robot_base_joint" type="fixed">
-    <parent link="base_footprint"/>
+    <parent link="base_footprint"/>  <!-- This was changed from world to base_link -->
     <child link="base_link"/>
     <origin xyz="0 0 ${wheel_radius}"/>
@@ -284,5 +284,10 @@
       <odom_publish_frequency>100</odom_publish_frequency>
       <topic>cmd_vel</topic>
+      <publish_odom>true</publish_odom>
+      <publish_wheel_tf>true</publish_wheel_tf>
+      <publish_odom_tf>true</publish_odom_tf>
       <odom_topic>odom</odom_topic>
+      <frame_id>odom</frame_id>
+      <child_frame_id>base_footprint</child_frame_id>
     </plugin>
     <!-- Joint state publisher -->

Commit message: Camera added

File: src/mobile_robot/model/flap_tb3_bot.xacro (robot description, xacro)
@@ -20,4 +20,8 @@
   <xacro:property name="lidar_length"        value="0.05"/>
   <xacro:property name="lidar_height_offset" value="${base_height/2.0 + 0.18}"/>
+  <!-- CAMERA (mount params) -->
+  <xacro:property name="camera_x_offset" value="${base_length/2 - 0.07}"/>
+  <xacro:property name="camera_z_offset" value="${base_height/2 + 0.12}"/>
+  <xacro:property name="camera_pitch"    value="0.18"/>
   <!-- Control -->
   <xacro:property name="max_linear_acceleration" value="10"/>
@@ -220,4 +224,66 @@
       <always_on>1</always_on>
       <visualize>true</visualize>
+    </sensor>
+  </gazebo>
+  <!-- ========================== -->
+  <!-- CAMERA (with optical frame) -->
+  <!-- ========================== -->
+  <joint name="camera_joint" type="fixed">
+    <parent link="base_link"/>
+    <child link="camera_link"/>
+    <origin xyz="${camera_x_offset} 0 ${camera_z_offset}" rpy="0 ${camera_pitch} 0"/>
+  </joint>
+  <link name="camera_link">
+    <visual>
+      <geometry>
+        <box size="0.010 0.03 0.03"/>
+      </geometry>
+      <material name="grey"/>
+    </visual>
+    <visual>
+      <origin xyz="0 0 -0.05" rpy="0 0 0"/>
+      <geometry>
+        <cylinder radius="0.002" length="0.1"/>
+      </geometry>
+      <material name="grey"/>
+    </visual>
+    <collision>
+      <geometry>
+        <box size="0.010 0.03 0.03"/>
+      </geometry>
+    </collision>
+    <inertial>
+      <origin xyz="0 0 0"/>
+      <mass value="0.10"/>
+      <inertia ixx="0.0002" iyy="0.0002" izz="0.0002" ixy="0" ixz="0" iyz="0"/>
+    </inertial>
+  </link>
+  <joint name="camera_optical_joint" type="fixed">
+    <parent link="camera_link"/>
+    <child link="camera_link_optical"/>
+    <origin xyz="0 0 0" rpy="${-pi/2} 0 ${-pi/2}"/>
+  </joint>
+  <link name="camera_link_optical"/>
+  <gazebo reference="camera_link">
+    <material>Gazebo/Grey</material>
+    <sensor name="camera" type="camera">
+      <pose>0 0 0 0 0 0</pose>
+      <visualize>true</visualize>
+      <update_rate>10</update_rate>
+      <camera>
+        <camera_info_topic>camera/camera_info</camera_info_topic>
+        <horizontal_fov>1.089</horizontal_fov>
+        <image>
+          <format>R8G8B8</format>
+          <width>640</width>
+          <height>480</height>
+        </image>
+        <clip>
+          <near>0.05</near>
+          <far>8.0</far>
+        </clip>
+      </camera>
+      <topic>camera/image_raw</topic>
+      <gz_frame_id>camera_link_optical</gz_frame_id>
     </sensor>
   </gazebo>
